File: timing.kicad_sch (KiCad schematic)
At the start: 13 parts, among them U11 CD74HC4040, U12 74LS20, U13 74LS20, U14 74LS30, U15 74LS30, U16 74LS00, U17 CD74HC4040, U18 74LS30, U19 74LS30, U20 74LS00, U3 74LS00, Y1 TFT660

Commit message: fix sync signal generation
Parts:
- added unit 2 of U13
- added U7: 74LS30, Package_SO:SOIC-14_3.9x8.7mm_P1.27mm, symbol 74xx:74LS30
Connections:
- net +5V: now also U7.11, U7.12, U7.6; no longer U15.12
- net HB12: now also U7.1; no longer U12.9
- net HB2: now also U7.2; no longer U12.10
- net HB3: now also U12.10, U12.12, U12.13, U12.9
- net HB4: now also U7.3; no longer U12.12
- net HB5: now also U7.4; no longer U12.13
- net VB2: now also U13.10, U13.12, U13.13, U13.9
- net at U12.8: now also U7.5; no longer U16.5
- new net: U16.5, U7.8
- new net: U13.8, U15.12
Other:
- note added: "Original Vsync Set Reset Q nQ(VSync) 600 1 1 0 1 601 1 0 1 0 602 1 1 1 0 603 1 0 1 0 604 1 1 1 0 605 0 0 x x 606 1 1 x x 607 0 0 x x"
- note added: "RST on line 628"
- note added: "Revised Vsync Set Reset Q nQ(VSync) 600 1 1 0 1 601 1 0 1 0 603 1 0 1 0 605 0 1 0 1 607 0 1 0 1 609 1 1 0 1 611 1 1 0 1 613 1 1 0 1"
- note added: "VSYNC start on line 601 end on line 605"
- note added: "~{VBlk} start on 600 end on 628"
- moved on the sheet: U12A, U12B, U13A, U14A, U15A, U16A, U16B, U16C, U16D, U18A, U19A, U20A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
