File: badVga.kicad_sch (KiCad schematic)
At the start: 32 parts, among them J1 VGA, SW1 SW_DIP_x04, U1 27C010, U12 74LS20, U13 74LS20, U14 74LS30, U15 74LS30, U16 74LS00, U18 74LS30, U19 74LS30, U2 74HC245, U20 74LS00, U21 IDT71342, U22 GAL16V8, U3 74LS00, U4 GAL16V8, U5 28C256, U6 74LS00, U8 74HC245

Commit message: improve rom use
Parts:
- removed JP1: ZWORKA, PCM_Jumper_AKL:Jumper_P2.54mm_D0.7mm, symbol Jumper:Jumper_2_Small_Open
- added R1, R15, R16, R2, R6, R7, R8: 10K, PCM_Resistor_SMD_AKL:R_0603_1608Metric, symbol Device:R_Small
- added R10, R11, R9: 20K, PCM_Resistor_SMD_AKL:R_0603_1608Metric, symbol Device:R_Small
- added R12, R13, R14: 100K, PCM_Resistor_SMD_AKL:R_0603_1608Metric, symbol Device:R_Small
- added R17, R18, R19, R20, R21, R22: 1K, PCM_Resistor_SMD_AKL:R_0603_1608Metric, symbol Device:R_Small
- added R23, R24, R25: 75R, PCM_Resistor_SMD_AKL:R_0603_1608Metric, symbol Device:R_Small
- added U10, U23, U24, U25, U7, U9: 74LVC1G3157, Package_SON:Texas_USON-6_1x1.45mm_P0.5mm_SMD, symbol 74xGxx:74LVC1G3157
- J1: footprint Library:CONN_AHDF15A-KG-TAXB_ASM -> Connector_Dsub:DSUB-15-HD_Socket_Horizontal_P2.29x2.54mm_EdgePinOffset8.35mm_Housed_MountingHolesOffset10.89mm
- SW1: value SW_DIP_x04 -> SW_DIP_x06; footprint Package_DIP:DIP-8_W7.62mm -> Button_Switch_THT:SW_DIP_SPSTx06_Slide_6.7x16.8mm_W7.62mm_P2.54mm_LowProfile; symbol Switch:SW_DIP_x04 -> Switch:SW_DIP_x06
- U12, U13: value 74LS20 -> 74HCT20
- U16, U20, U3, U6: value 74LS00 -> 74HCT00
- U2, U8: value 74HC245 -> 74HCT245
Connections:
- net +5V: now also SW1.1, SW1.2, SW1.3, SW1.5, SW1.6, R12.1, R13.1, R14.1, U10.5 (VCC), U23.5 (VCC), U24.5 (VCC), U25.5 (VCC), U7.5 (VCC), U9.5 (VCC)
- net BLUE: now also SW1.10, R2.2, U25.6; no longer J1.3, SW1.6
- net CP438: now also SW1.7
- net GND: now also R1.2, R15.1, R16.1, R17.2, R18.2, R19.2, R2.1, R20.2, R21.2, R22.2, R23.2, R24.2, R25.2, U10.2 (GND), U23.1, U23.2 (GND), U24.1, U24.2 (GND), U25.1, U25.2 (GND), U7.2 (GND), U9.2 (GND)
- net GREEN: now also SW1.11, R15.2, U24.6; no longer J1.2, SW1.7
- net INV: now also SW1.9; no longer SW1.5
- net RED: now also SW1.12, R16.2, U23.6; no longer J1.1, SW1.8
- net pixel: now also U23.3, U24.3, U25.3; no longer SW1.1, SW1.2, SW1.3
- net at U1.15 (D2): now also R17.1, R6.1
- net at U1.17 (D3): now also R18.1, R9.1
- net at U1.18 (D4): now also R19.1, R7.1
- net at U1.19 (D5): now also R10.1, R20.1
- net at U1.20 (D6): now also R21.1, R8.1
- net at U1.21 (D7): now also R11.1, R22.1
- new net: U10.3, U25.4
- new net: U23.4, U7.3
- new net: U24.4, U9.3
- new net BLUE2: R11.2, R14.2, R8.2, U10.1
- new net COLOUR: R1.1, SW1.8, U10.6, U7.6, U9.6
- new net GREEN2: R10.2, R13.2, R7.2, U9.1
- new net RED2: R12.2, R6.2, R9.2, U7.1
- new net xBLUE: J1.3, R23.1, U10.4
- new net xGREEN: J1.2, R24.1, U9.4
- new net xRED: J1.1, R25.1, U7.4
- no-connect marks 28 -> 23
Other:
- moved on the sheet: C1, C2, C3, C4, C5, C6, C7, C8, C9, R3, R4, R5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

Commit message: fix sync signals
Parts:
- removed unit 2 of U13
- added C10: 10nF, Capacitor_SMD:C_0805_2012Metric, symbol Device:C_Small
- added U26: 74LS30, Package_SO:SOIC-14_3.9x8.7mm_P1.27mm, symbol 74xx:74LS30
- U10, U23, U24, U25, U7, U9: LCSC (none) -> C548323
Connections:
- net +5V: now also C10.1, U26.14 (VCC)
- net GND: now also C10.2, U26.7 (GND)
- no-connect marks 23 -> 22
